Commit message: Implement grasping with the gripper

File: urdf/gripper.urdf.xacro (robot description, xacro)
@@ -16,12 +16,31 @@
                         </geometry>
                 </visual>
+        </link>
+        <joint name="finger_left_joint" type="prismatic">
+                <origin xyz="0 0 0" rpy="0 0 0"/>
+                <axis xyz="0 1 0" />
+                <limit upper="0" lower="0" velocity="0" effort="0"/>
+                <parent link="gripper"/>
+                <child link="finger_left"/>
+        </joint>
+        <link name="finger_left">
                 <visual name="visual">
-                        <origin xyz="0 0.075 ${-0.05 -0.05}" rpy="0 0 0" />
+                        <origin xyz="0 0 -0.1" rpy="0 0 0" />
                         <geometry>
                                 <box size="0.02 0.02 0.1"/>
                         </geometry>
                 </visual>
+        </link>
+        <joint name="finger_right_joint" type="prismatic">
+                <origin xyz="0 0 0" rpy="0 0 0"/>
+                <axis xyz="0 1 0" />
+                <limit upper="0" lower="0" velocity="0" effort="0"/>
+                <mimic joint="finger_left_joint" multiplier="-1" />
+                <parent link="gripper"/>
+                <child link="finger_right"/>
+        </joint>
+        <link name="finger_right">
                 <visual name="visual">
-                        <origin xyz="0 -0.075 ${-0.05 -0.05}" rpy="0 0 0" />
+                        <origin xyz="0 0 -0.1" rpy="0 0 0" />
                         <geometry>
                                 <box size="0.02 0.02 0.1"/>
