Commit message: Add end-effector link for control
This is now compatible with `arne_motion_simulator`'s control link.

File: urdf/aria_v2.urdf.xacro (robot description, xacro)
@@ -8,3 +8,10 @@
     <origin xyz="0 0 0" rpy="0 0 0" />
   </joint>
+  <!-- This is the link for direct control and skill replay -->
+  <link name="control" />
+  <joint name="control_joint" type="fixed">
+    <parent link="eef_link" />
+    <child link="control" />
+    <origin xyz="0 0 0" rpy="0 ${pi/2} ${pi/2}" />
+  </joint>
 </robot>
